File: hardware/KungFuFlash2.kicad_pcb (KiCad board)
At the start: 2 copper layers, 60.6 x 62 mm, 55 parts, among them J1 SWD, J3 Wifi, J4 USB_C_Receptacle_USB2.0, Q1 BC817, SW1 Reset, SW2 Menu, SW3 Special, U1 C64-Exp-Port, U2 AMS1117-3.3, U3 STM32H7B0VBTx, Y1 25 MHz

Commit message: fix: rename J4 to J2, move label for R17, update URL of repo
Parts:
- renumbered J4 to J2
Other:
- board text added: "Kung Fu Flash 2"
- board text added: "Rev. 2"
- board text added: "codeberg.org/KimJorgensen/KungFuFlash2"
- board text removed: "Rev. 1"
- board text removed: "github.com/KimJorgensen/KungFuFlash2"
- board text removed: "locked"
