File: hardware/KungFuFlash2.kicad_pcb (KiCad board)
At the start: 2 copper layers, 60.6 x 62 mm, 55 parts, among them J1 SWD, J2 USB_C_Receptacle_USB2.0, J3 Wifi, Q1 BC817, SW1 Reset, SW2 Menu, SW3 Special, U1 C64-Exp-Port, U2 AMS1117-3.3, U3 STM32H7B0VBTx, Y1 25 MHz

Commit message: feat: update symbol table fields with BOM information for production
Changed lines of the file:
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@@
 		)
 		(sheetfile "KungFuFlash2.kicad_sch")
-		(attr through_hole)
+		(attr through_hole exclude_from_pos_files exclude_from_bom)
 		(duplicate_pad_numbers_are_jumpers no)
 		(fp_line
@@
 		(tags "USB C Type-C Receptacle SMD")
 		(property "Reference" "J2"
-			(at 0 -5.715 90)
+			(at 0 2.2 90)
 			(layer "F.SilkS")
 			(effects
@@
 	)
 	(gr_text "GND"
-		(at 122.742 86.995 0)
+		(at 130.175 100.457 0)
 		(layer "F.SilkS")
 		(effects
@@
 		)
 	)
-	(gr_text "TX"
-		(at 123.19 84.455 0)
+	(gr_text "CLK"
+		(at 130.429 105.537 0)
 		(layer "F.SilkS")
 		(effects
@@
 		)
 	)
-	(gr_text "GND"
-		(at 130.175 100.457 0)
+	(gr_text "DIO"
+		(at 130.556 102.995 0)
 		(layer "F.SilkS")
 		(effects
@@
 		)
 	)
-	(gr_text "CLK"
-		(at 130.429 105.537 0)
+	(gr_text "B0"
+		(at 130.683 95.377 0)
 		(layer "F.SilkS")
 		(effects
@@
 		)
 	)
-	(gr_text "DIO"
-		(at 130.556 102.87 0)
+	(gr_text "3.3"
+		(at 130.683 97.917 0)
 		(layer "F.SilkS")
 		(effects
@@
 		)
 	)
-	(gr_text "B0"
-		(at 130.683 95.377 0)
+	(gr_text "Rev. 2"
+		(at 79.6036 96.4184 0)
 		(layer "F.SilkS")
 		(effects
@@
 				(size 1 1)
 				(thickness 0.25)
-				(bold yes)
 			)
-			(justify left)
 		)
 	)
-	(gr_text "3.3"
-		(at 130.683 97.917 0)
+	(gr_text "TX"
+		(at 123.675 85.35 90)
 		(layer "F.SilkS")
 		(effects
@@
 		)
 	)
-	(gr_text "Rev. 2"
-		(at 79.6036 96.4184 0)
+	(gr_text "GND"
+		(at 123.692 88.75 90)
 		(layer "F.SilkS")
 		(effects
@@
 				(size 1 1)
 				(thickness 0.25)
+				(bold yes)
 			)
+			(justify left)
 		)
 	)
