File: hardware/KungFuFlash2.kicad_sch (KiCad schematic)
At the start: 54 parts, among them J1 SWD, J3 Wifi, J4 USB_C_Receptacle_USB2.0, Q1 BC817, SW1 Reset, SW2 Menu, SW3 Special, U1 C64-Exp-Port, U2 AMS1117-3.3, U3 STM32H7B0VBTx, Y1 25 MHz

Commit message: fix: update schematic revision and export new PDF
Parts:
- TP1, TP2, TP3: value ~ -> (none)

Commit message: feat: update symbol table fields with BOM information for production
Parts:
- C1, C2: LCSC Part# (none) -> C318691; Manf (none) -> Samsung Electro-Mechanics; Manf# (none) -> CL21A106KAYNNNG
- C10, C13, C14, C15, C16, C17, C18, C19, C3, C4, C5, C6, C9: LCSC Part# (none) -> C1591; Manf (none) -> Samsung Electro-Mechanics; Manf# (none) -> CL10B104KB8NNNC
- C11, C12: LCSC Part# (none) -> C5362585; Manf (none) -> Samsung Electro-Mechanics; Manf# (none) -> CL21B225KBYVPNE
- C7, C8: LCSC Part# (none) -> C346210; Manf (none) -> Samsung Electro-Mechanics; Manf# (none) -> CL10C200JB81PNC
- D1: value LED -> Green; LCSC Part# (none) -> C2297; Manf (none) -> Hubei KENTO Elec; Manf# (none) -> KT-0805G
- D2, D3: LCSC Part# (none) -> C64998; Manf (none) -> MDD; Manf# (none) -> SS33
- J1: value SWD -> DNP; LCSC Part# (none) -> DNP; Manf (none) -> DNP; Manf# (none) -> DNP; now not fitted
- J2: renamed from J4; LCSC Part# (none) -> C165948; Manf (none) -> Korean Hroparts Elec; Manf# (none) -> TYPE-C-31-M-12
- J3: value Wifi -> DNP; LCSC Part# (none) -> DNP; Manf (none) -> DNP; Manf# (none) -> DNP; now not fitted
- Q1: value BC817 -> BC817-40; LCSC Part# (none) -> C916383; Manf (none) -> JSMSEMI; Manf# (none) -> BC817
- R1, R4, R5, R6, R7: LCSC Part# (none) -> C139861; Manf (none) -> FH; Manf# (none) -> RS-05K5100FT
- R10, R11, R12, R13, R14, R15, R8, R9: LCSC Part# (none) -> C115424; Manf (none) -> FH; Manf# (none) -> RS-05K1000FT
- R16, R17: LCSC Part# (none) -> C118848; Manf (none) -> FH; Manf# (none) -> RS-05K5101FT
- R2, R3: LCSC Part# (none) -> C115309; Manf (none) -> FH; Manf# (none) -> RS-05K1002FT
- SW1: value Reset -> Tactile Switch SPST 250gf 5mm PC Pin 6mm x 6mm Through Hole; LCSC Part# (none) -> C42416245; Manf (none) -> SHOU HAN; Manf# (none) -> SH-6X6X5H-CJ
- SW2: value Menu -> Tactile Switch SPST 250gf 5mm PC Pin 6mm x 6mm Through Hole; LCSC Part# (none) -> C42416245; Manf (none) -> SHOU HAN; Manf# (none) -> SH-6X6X5H-CJ
- SW3: value Special -> Tactile Switch SPST 250gf 5mm PC Pin 6mm x 6mm Through Hole; LCSC Part# (none) -> C42416245; Manf (none) -> SHOU HAN; Manf# (none) -> SH-6X6X5H-CJ
- TP1, TP2, TP3: LCSC Part# (none) -> DNP; Manf (none) -> DNP; Manf# (none) -> DNP; now left out of the parts list
- U1: value C64-Exp-Port -> Edge Connector, Immersion gold (1U"), Bevelling 45°; LCSC Part# (none) -> DNP; Manf (none) -> DNP; Manf# (none) -> DNP; now left out of the parts list
- U2: LCSC Part# (none) -> C6186; Manf (none) -> Advanced Monolithic Systems; Manf# (none) -> AMS1117-3.3
- U3: LCSC Part# (none) -> C730227; Manf (none) -> ST; Manf# (none) -> STM32H7B0VBT6
- XS1: LCSC Part# (none) -> C111196; Manf ebay -> SOFNG; Manf# _ -> TF-15x15
- Y1: LCSC Part# (none) -> C9006; Manf (none) -> YXC Crystal Oscillators; Manf# (none) -> X322525MOB4SI
